Commit message: added starter files.

File: inv_kin/urdf/simple_robot.xacro (robot description, xacro)
@@ -1,73 +1,2 @@
-<?xml version="1.0"?>
-<robot xmlns:xacro="http://www.ros.org/wiki/xacro" name="simple_robot">
-  <!-- Materials -->
-  <material name="red">
-    <color rgba="1 0 0 1"/>
-  </material>
-  <material name="green">
-    <color rgba="0 1 0 1"/>
-  </material>
-  <material name="blue">
-    <color rgba="0 0 1 1"/>
-  </material>
-  <!-- World -->
-  <link name="world"/>
-  <!-- Joint 1 -->
-  <joint name="joint1" type="revolute">
-    <parent link="world"/>
-    <child link="link1"/>
-    <origin xyz="0 0 0" rpy="0 0 0"/>
-    <axis xyz="0 0 1"/>
-    <limit lower="-${pi}" upper="${pi}" effort="1" velocity="${pi}"/>
-  </joint>
-  <!-- Link 1 -->
-  <link name="link1">
-    <visual>
-      <geometry>
-        <mesh filename="package://simple_robot/meshes/link1.stl"/>
-      </geometry>
-      <material name="red"/>
-    </visual>
-  </link>
-  <!-- Joint 2 -->
-  <joint name="joint2" type="revolute">
-    <parent link="link1"/>
-    <child link="link2"/>
-    <origin xyz="-0.100 0 0" rpy="0 -${pi/2} 0"/>
-    <axis xyz="0 0 1"/>
-    <limit lower="-${pi}" upper="${pi}" effort="1" velocity="${pi}"/>
-  </joint>
-  <!-- link 2 -->
-  <link name="link2">
-    <visual>
-      <geometry>
-        <mesh filename="package://simple_robot/meshes/link2.stl"/>
-      </geometry>
-      <material name="green"/>
-    </visual>
-  </link>
-  <!-- Joint 3 -->
-  <joint name="joint3" type="prismatic">
-    <parent link="link2"/>
-    <child link="link3"/>
-    <origin xyz="0 0.200 0.100" rpy="-${pi/2} 0 0"/>
-    <axis xyz="0 0 1"/>
-    <limit lower="0" upper="0.150" effort="1" velocity="100"/>
-  </joint>
-  <!-- link 3 -->
-  <link name="link3">
-    <visual>
-      <geometry>
-        <mesh filename="package://simple_robot/meshes/link3.stl"/>
-      </geometry>
-      <material name="blue"/>
-    </visual>
-  </link>
-  <link name="ee_link"/>
-  <!-- Fixed EE joint -->
-  <joint name="ee_joint" type="fixed">
-    <parent link="link3"/>
-    <child link="ee_link"/>
-    <origin xyz="0 0 0.225" rpy="${pi/2} 0 ${pi/2}"/>
-  </joint>
-</robot>
+<!-- DEFINE YOUR URDF HERE -->
+<!-- USE YOUR PREVIOUS TAKE-HOME ASSIGNMENT SOLUTION AS A STARTING PLACE -->
